File: cad/electronics/myrt-charging_stations.kicad_sch (KiCad schematic)
At the start: 20 parts, among them P10 OUT, P11 OUT, P3 IN, P5 OUT, P6 IN, P7 IN, P8 IN, P9 OUT

Commit message: Updated source names to match with other documents (slow/medium/fast)
Other:
- note added: "Fast source (5V, 150mA max, R:33Ω)"
- note added: "Medium source (5V, 50mA max, R:100Ω)"
- note added: "Slow Source (5V, 10mA max, R:500Ω)"
- note removed: "Fast source (5V, 150mA max)"
- note removed: "Medium source (5V, 50mA max)"
- note removed: "Regular Source (5V, 10mA max, R:500Ω)"
- note removed: "Regular charging station (10mA)"
