File: cad/electronics/myrt.kicad_pcb (KiCad board)
At the start: 2 copper layers, 105.4 x 203.3 mm, 55 parts, among them J1 Spare1, J10 Spare3, J11 Spare4, J2 Spare2, J3 Regular, J4 Regular, J6 USB_B PTH Receptable, J7 Serial 7 Segment Display, J8 Accelerated, J9 Fast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

Commit message: Corrected error "Expecting pts" on openning the Kicad PCB file (corrupted file)
Routing:
- net /Charging stations/POWER_GND_S4: track 7.49 -> 0.00 mm, vias 1 -> 0
- net /Charging stations/POWER_GND_S1: track 7.49 -> 0.00 mm, vias 1 -> 0
